File: sch/mplayer/v0.01/sdmplayerv0.01.kicad_pcb (KiCad board)
At the start: 2 copper layers, 47.2 x 69.6 mm, 6 parts, among them CON1 SD_Card, P1 USB_OTG, P2 CONN_01X09, U1 VS1053, U2 TP4056, U3 STM32F103RCTx

Commit message: player_scheme_0.01
Parts:
- added C1: 22pF, Capacitors_SMD:C_0402, F.Cu at (161.5, 127.5)
- added C2: 22pF, Capacitors_SMD:C_0402, F.Cu at (157.0, 106.2)
- added C3: 22pF, Capacitors_SMD:C_0402, F.Cu at (161.5, 122.4)
- added C4: 22pF, Capacitors_SMD:C_0402, F.Cu at (159.0, 131.1)
- added C5: 100nF, Capacitors_SMD:C_0402, F.Cu at (171.2, 125.0)
- added C6: 33pF, Capacitors_SMD:C_0805_HandSoldering, F.Cu at (179.3, 130.6)
- added C7: 33pF, Capacitors_SMD:C_0805_HandSoldering, F.Cu at (170.2, 137.2)
- added C8: 1uF, Capacitors_SMD:C_0805_HandSoldering, F.Cu at (164.1, 150.9)
- added IC1: AT24CS64-SSHM, Housings_SOIC:SOIC-8-1EP_3.9x4.9mm_Pitch1.27mm, F.Cu at (150.9, 118.4)
- added P3: ClockBat, Pin_Headers:Pin_Header_Straight_1x01, F.Cu at (147.8, 126.5)
- added P4: USART1, Pin_Headers:Pin_Header_Straight_1x02, F.Cu at (188.5, 138.7)
- added P5: AudioJack, Pin_Headers:Pin_Header_Straight_1x03, F.Cu at (145.8, 142.2)
- added R1: R, Resistors_SMD:R_0603_HandSoldering, F.Cu at (151.4, 111.8)
- added R2: R, Resistors_SMD:R_0603_HandSoldering, F.Cu at (157.5, 117.3)
- added R3: 5k, Resistors_SMD:R_0603_HandSoldering, F.Cu at (156.5, 111.3)
- added R4: R, Resistors_SMD:R_0603_HandSoldering, F.Cu at (166.1, 131.6)
- added R5: 1M, Resistors_SMD:R_0603_HandSoldering, F.Cu at (173.2, 141.2)
- added R6: 100k, Resistors_SMD:R_0603_HandSoldering, F.Cu at (174.2, 151.9)
- added SW1: SW_PUSH, Pin_Headers:Pin_Header_Angled_1x02, F.Cu at (145.8, 107.7)
- added Y1: 12.288MHz, Crystals:Crystal_SMD_0603_4Pads, F.Cu at (178.8, 141.2)
- added Y2: 8MHz, Crystals:Crystal_SMD_0603_4Pads, F.Cu at (165.1, 127.5)
- added Y3: 32768Hz, Crystals:Crystal_SMD_0603_4Pads, F.Cu at (157.5, 127.5)
- CON1: footprint Connect:SD_Card_Receptacle -> Housings_SOIC:SOIC-14_3.9x8.7mm_Pitch1.27mm
- moved CON1 77.7 mm to (148.8, 93.5), turned to 90 degrees
- moved P2 60.6 mm to (189.0, 117.3), turned to 180 degrees
- moved U2 41.0 mm to (172.7, 100.1)
- moved U3 9.14 mm to (167.1, 115.3), turned to 90 degrees
- moved U1 7.13 mm to (163.6, 140.2), turned to 90 degrees
- moved P1 1.44 mm to (184.9, 154.4)
Connections:
- net Net-(P1-Pad1) renamed +5V
- CON1 pad 1: Net-(CON1-Pad1) -> /DAT3
- CON1 pad 10: Net-(CON1-Pad10) -> /SD_CONN
- CON1 pad 12: Net-(CON1-Pad12) -> GND
- CON1 pad 13: Net-(CON1-Pad13) -> GND
- CON1 pad 2: Net-(CON1-Pad2) -> /SD_CMD
- CON1 pad 3: Net-(CON1-Pad3) -> GND
- CON1 pad 4: Net-(CON1-Pad4) -> +3V3
- CON1 pad 5: Net-(CON1-Pad5) -> /SD_CLK
- CON1 pad 6: Net-(CON1-Pad6) -> GND
- CON1 pad 7: Net-(CON1-Pad7) -> /DAT0
- CON1 pad 8: Net-(CON1-Pad8) -> /DAT1
- CON1 pad 9: Net-(CON1-Pad9) -> /DAT2
- P1 pad 2: Net-(P1-Pad2) -> /USB_DM
- P1 pad 3: Net-(P1-Pad3) -> /USB_DP
- P1 pad 5: Net-(P1-Pad5) -> GND
- P2 pad 1: Net-(P2-Pad1) -> +3V3
- P2 pad 2: Net-(P2-Pad2) -> GND
- P2 pad 3: Net-(P2-Pad3) -> /PC4
- P2 pad 4: Net-(P2-Pad4) -> /PC5
- P2 pad 5: Net-(P2-Pad5) -> /PB2
- P2 pad 6: Net-(P2-Pad6) -> /PB1
- P2 pad 7: Net-(P2-Pad7) -> /PB0
- P2 pad 8: Net-(P2-Pad8) -> /I2C2_SCL
- P2 pad 9: Net-(P2-Pad9) -> /I2C2_SDA
- U1 pad 10: Net-(U1-Pad10) -> Net-(R6-Pad1)
- U1 pad 11: Net-(U1-Pad11) -> Net-(R6-Pad1)
- U1 pad 12: Net-(U1-Pad12) -> Net-(R6-Pad1)
- U1 pad 13: Net-(U1-Pad13) -> /xDCS
- U1 pad 14: Net-(U1-Pad14) -> +3V3
- U1 pad 16: Net-(U1-Pad16) -> GND
- U1 pad 19: Net-(U1-Pad19) -> +3V3
- U1 pad 20: Net-(U1-Pad20) -> GND
- U1 pad 21: Net-(U1-Pad21) -> GND
- U1 pad 22: Net-(U1-Pad22) -> GND
- U1 pad 23: Net-(U1-Pad23) -> /xCS
- U1 pad 24: Net-(U1-Pad24) -> +1V8
- U1 pad 25: Net-(U1-Pad25) -> Net-(R6-Pad1)
- U1 pad 26: Net-(U1-Pad26) -> +3V3
- U1 pad 28: Net-(U1-Pad28) -> /SPI2_SCK
- U1 pad 29: Net-(U1-Pad29) -> /SPI2_MOSI
- U1 pad 3: Net-(U1-Pad3) -> /xRST
- U1 pad 30: Net-(U1-Pad30) -> /SPI2_MISO
- U1 pad 31: Net-(U1-Pad31) -> +1V8
- U1 pad 33: Net-(U1-Pad33) -> Net-(R6-Pad1)
- U1 pad 34: Net-(U1-Pad34) -> Net-(R6-Pad1)
- U1 pad 35: Net-(U1-Pad35) -> GND
- U1 pad 36: Net-(U1-Pad36) -> Net-(R6-Pad1)
- U1 pad 37: Net-(U1-Pad37) -> GND
- U1 pad 38: Net-(U1-Pad38) -> +3V3
- U1 pad 4: Net-(U1-Pad4) -> GND
- U1 pad 40: Net-(U1-Pad40) -> GND
- U1 pad 41: Net-(U1-Pad41) -> GND
- U1 pad 43: Net-(U1-Pad43) -> +3V3
- U1 pad 45: Net-(U1-Pad45) -> +3V3
- U1 pad 47: Net-(U1-Pad47) -> GND
- U1 pad 5: Net-(U1-Pad5) -> +1V8
- U1 pad 6: Net-(U1-Pad6) -> +3V3
- U1 pad 7: Net-(U1-Pad7) -> +1V8
- U1 pad 8: Net-(U1-Pad8) -> /DREQ
- U1 pad 9: Net-(U1-Pad9) -> Net-(R6-Pad1)
- U3 pad 12: Net-(U3-Pad12) -> GND
- U3 pad 13: Net-(U3-Pad13) -> +3V3
- U3 pad 18: Net-(U3-Pad18) -> GND
- U3 pad 19: Net-(U3-Pad19) -> +3V3
- U3 pad 22: Net-(U3-Pad22) -> /xDCS
- U3 pad 24: Net-(U3-Pad24) -> /PC4
- U3 pad 25: Net-(U3-Pad25) -> /PC5
- U3 pad 26: Net-(U3-Pad26) -> /PB0
- U3 pad 27: Net-(U3-Pad27) -> /PB1
- U3 pad 28: Net-(U3-Pad28) -> /PB2
- U3 pad 29: Net-(U3-Pad29) -> /I2C2_SCL
- U3 pad 30: Net-(U3-Pad30) -> /I2C2_SDA
- U3 pad 31: Net-(U3-Pad31) -> GND
- U3 pad 32: Net-(U3-Pad32) -> +3V3
- U3 pad 33: Net-(U3-Pad33) -> /xRST
- U3 pad 34: Net-(U3-Pad34) -> /SPI2_SCK
- U3 pad 35: Net-(U3-Pad35) -> /SPI2_MISO
- U3 pad 36: Net-(U3-Pad36) -> /SPI2_MOSI
- U3 pad 37: Net-(U3-Pad37) -> /DREQ
- U3 pad 38: Net-(U3-Pad38) -> /xCS
- U3 pad 39: Net-(U3-Pad39) -> /DAT0
- U3 pad 40: Net-(U3-Pad40) -> /DAT1
- U3 pad 44: Net-(U3-Pad44) -> /USB_DM
- U3 pad 45: Net-(U3-Pad45) -> /USB_DP
- U3 pad 47: Net-(U3-Pad47) -> GND
- U3 pad 48: Net-(U3-Pad48) -> +3V3
- U3 pad 50: Net-(U3-Pad50) -> /SD_CONN
- U3 pad 51: Net-(U3-Pad51) -> /DAT2
- U3 pad 52: Net-(U3-Pad52) -> /DAT3
- U3 pad 53: Net-(U3-Pad53) -> /SD_CLK
- U3 pad 54: Net-(U3-Pad54) -> /SD_CMD
- U3 pad 58: Net-(U3-Pad58) -> /I2C1_SCL
- U3 pad 59: Net-(U3-Pad59) -> /I2C1_SDA
- U3 pad 60: Net-(U3-Pad60) -> GND
- U3 pad 63: Net-(U3-Pad63) -> GND
- U3 pad 64: Net-(U3-Pad64) -> +3V3

Commit message: fix
Parts:
- added C10: 10uF, Capacitors_SMD:C_0805_HandSoldering, F.Cu at (246.1, 117.2)
- added C11: 1uF, Capacitors_SMD:C_0805_HandSoldering, F.Cu at (260.5, 99.3)
- added C12: 0.47uF, Capacitors_SMD:C_0805_HandSoldering, F.Cu at (253.8, 107.5)
- added C13: 0.1uF, Capacitors_SMD:C_1206_HandSoldering, F.Cu at (247.1, 110.7)
- added C14: 0.1uF, Capacitors_SMD:C_1206_HandSoldering, F.Cu at (254.5, 101.0)
- added C15: C, Capacitors_SMD:C_1206_HandSoldering, F.Cu at (231.8, 123.1)
- added C16: 0.1uF, Capacitors_SMD:C_1206_HandSoldering, F.Cu at (261.3, 92.8)
- added C17: 0.1uF, Capacitors_SMD:C_1206_HandSoldering, F.Cu at (231.8, 116.4)
- added C18: 0.1uF, Capacitors_SMD:C_1206_HandSoldering, F.Cu at (240.0, 111.7)
- added C9: 4.7uF, Capacitors_SMD:C_0805_HandSoldering, F.Cu at (224.1, 129.2)
- added L1: 2.2uH, Capacitors_SMD:C_0805_HandSoldering, F.Cu at (229.1, 129.6)
- added P6: LiPo battery, Socket_Strips:Socket_Strip_Straight_1x02, F.Cu at (252.9, 95.6)
- added R10: 18.2k, Resistors_SMD:R_0603_HandSoldering, F.Cu at (256.1, 119.5)
- added R11: 100k, Resistors_SMD:R_0603_HandSoldering, F.Cu at (242.8, 129.2)
- added R12: 4.7k, Resistors_SMD:R_0603_HandSoldering, F.Cu at (233.9, 130.6)
- added R13: 4.7k, Resistors_SMD:R_0603_HandSoldering, F.Cu at (251.7, 125.4)
- added R14: 100, Resistors_SMD:R_0603_HandSoldering, F.Cu at (265.3, 104.6)
- added R15: 100, Resistors_SMD:R_0603_HandSoldering, F.Cu at (261.8, 116.4)
- added R16: 0.01, Resistors_SMD:R_0603_HandSoldering, F.Cu at (247.2, 129.2)
- added R7: 1k, Resistors_SMD:R_0603_HandSoldering, F.Cu at (247.1, 123.3)
- added R8: 2k, Resistors_SMD:R_0603_HandSoldering, F.Cu at (251.5, 119.5)
- added R9: 1.8M, Resistors_SMD:R_0603_HandSoldering, F.Cu at (264.7, 110.5)
- added U4: BQ24090, Housings_SSOP:MSOP-10-1EP_3x3mm_Pitch0.5mm, F.Cu at (217.9, 129.7)
- added U5: BQ27510, Housings_SSOP:MSOP-12-1EP_3x4mm_Pitch0.65mm, F.Cu at (247.3, 103.2)
- U2: value TP4056 -> LM3671MF-3.3; footprint SMD_Packages:SO-8_PowerPAK_Vishay_Single -> TO_SOT_Packages_SMD:SOT-23-5
- moved R4 106.1 mm to (267.0, 98.7)
- moved C2 105.4 mm to (261.2, 122.1)
- moved R3 103.9 mm to (260.2, 105.4), turned to 0 degrees
- moved R1 101.5 mm to (252.9, 113.6)
- moved P5 97.0 mm to (230.8, 95.6), turned to 0 degrees
- moved C6 95.8 mm to (267.3, 92.6)
- moved P3 94.4 mm to (240.1, 106.3)
- moved Y3 93.1 mm to (244.5, 94.3)
- moved R6 91.5 mm to (257.3, 113.6)
- moved R2 85.3 mm to (242.6, 123.3), turned to 0 degrees
- moved C5 85.3 mm to (256.5, 125.2)
- moved C8 80.7 mm to (237.9, 118.2)
- moved U1 72.5 mm to (221.4, 96.5), turned to 0 degrees
- moved CON1 71.6 mm to (218.5, 109.9), turned to 0 degrees
- moved C4 70.0 mm to (224.5, 106.3)
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Connections:
- U2 pad 1: Net-(U2-Pad1) -> +BATT
- U2 pad 2: Net-(U2-Pad2) -> GND
- U2 pad 3: Net-(U2-Pad3) -> +BATT
- U2 pad 4: Net-(U2-Pad4) -> +3V3
- U3 pad 10: Net-(U3-Pad10) -> /PC2
- U3 pad 11: Net-(U3-Pad11) -> /PC3
- U3 pad 23: Net-(U3-Pad23) -> /PA7
- U3 pad 42: Net-(U3-Pad42) -> Net-(P4-Pad1)
- U3 pad 43: Net-(U3-Pad43) -> Net-(P4-Pad2)
- U3 pad 8: Net-(U3-Pad8) -> /PC0
- U3 pad 9: Net-(U3-Pad9) -> /PC1

Commit message: layout upd
Parts:
- removed R4: R, Resistors_SMD:R_0603_HandSoldering
- added C19: 10uF, Capacitors_SMD:C_0805_HandSoldering, F.Cu at (179.8, 136.1)
- added C20: 100nF, Capacitors_SMD:C_0402, F.Cu at (166.3, 106.1)
- added C21: 100nF, Capacitors_SMD:C_0402, F.Cu at (153.9, 123.9)
- added C22: 100nF, Capacitors_SMD:C_0402, F.Cu at (163.8, 118.1)
- added C23: 100nF, Capacitors_SMD:C_0402, F.Cu at (158.4, 135.3)
- added C24: 100nF, Capacitors_SMD:C_0402, F.Cu at (163.8, 119.4)
- added C25: 100nF, Capacitors_SMD:C_0402, F.Cu at (156.5, 111.3)
- added C26: 100nF, Capacitors_SMD:C_0402, F.Cu at (165.0, 102.6)
- added C27: 100nF, Capacitors_SMD:C_0402, F.Cu at (167.6, 138.9)
- added C28: 100nF, Capacitors_SMD:C_0402, F.Cu at (155.1, 104.9)
- added C29: 100nF, Capacitors_SMD:C_0402, F.Cu at (173.2, 128.3)
- added C30: 100nF, Capacitors_SMD:C_0402, F.Cu at (162.0, 124.6)
- added C31: 100nF, Capacitors_SMD:C_0402, F.Cu at (149.3, 118.5)
- added C32: 100nF, Capacitors_SMD:C_0402, F.Cu at (150.9, 116.3)
- added U6: NCP1117ST18T3G, TO_SOT_Packages_SMD:SOT-223, F.Cu at (148.3, 124.0)
- C10, C9, IC1, R10, R11, R12, R13, R14, R15, R7, R8, R9, U4: moved to B.Cu
- C11: footprint Capacitors_SMD:C_0805_HandSoldering -> Capacitors_SMD:C_0603_HandSoldering; moved to B.Cu
- C13, C14, C16, C17, C18: footprint Capacitors_SMD:C_1206_HandSoldering -> Capacitors_SMD:C_0402; moved to B.Cu
- C15: value C -> 1uF; footprint Capacitors_SMD:C_1206_HandSoldering -> Capacitors_SMD:C_0603_HandSoldering
- C8: footprint Capacitors_SMD:C_0805_HandSoldering -> Capacitors_SMD:C_0603_HandSoldering
- CON1: footprint Housings_SOIC:SOIC-14_3.9x8.7mm_Pitch1.27mm -> v0:Micro_SD_card_slot; moved to B.Cu
- L1: footprint Capacitors_SMD:C_0805_HandSoldering -> Inductors:self_cms_we-tpc_XL
- SW1: footprint Pin_Headers:Pin_Header_Angled_1x02 -> Pin_Headers:Pin_Header_Straight_1x02
- U5: footprint Housings_SSOP:MSOP-12-1EP_3x4mm_Pitch0.65mm -> v0:SON-12; moved to B.Cu
- Y1, Y2: footprint Crystals:Crystal_SMD_0603_4Pads -> Crystals:Crystal_HC49-SD_SMD
- Y3: footprint Crystals:Crystal_SMD_0603_4Pads -> v0:KX-327S
- moved C6 116.7 mm to (152.0, 110.6)
- moved C2 111.4 mm to (151.3, 140.3)
- moved R9 107.8 mm to (163.2, 146.7), turned to 90 degrees
- moved C12 102.6 mm to (151.3, 102.9), turned to 90 degrees
- moved R1 100.0 mm to (155.0, 134.2), turned to 90 degrees
- moved R14 99.8 mm to (171.9, 139.6)
- moved P6 99.2 mm to (174.9, 157.0), turned to 180 degrees
- moved U5 98.4 mm to (162.3, 152.8)
- moved C16 98.2 mm to (173.3, 136.4), turned to 270 degrees
- moved R15 95.6 mm to (173.8, 153.8), turned to 180 degrees
- moved R10 92.7 mm to (168.3, 149.1), turned to 180 degrees
- moved C14 92.3 mm to (172.4, 143.3), turned to 90 degrees
- moved C5 92.1 mm to (165.4, 138.9)
- moved R2 90.3 mm to (153.0, 134.2), turned to 90 degrees
- moved C11 90.1 mm to (182.1, 143.4), turned to 270 degrees
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Connections:
- U1 pad 32: Net-(R4-Pad1) -> +3V3

Commit message: upd
Parts:
- added REF**: 1pin, Connect:1pin, F.Cu at (188.0, 124.5)
- added REF**: 1pin, Connect:1pin, F.Cu at (188.0, 92.5)
- added REF**: 1pin, Connect:1pin, F.Cu at (188.0, 156.0)
- added REF**: 1pin, Connect:1pin, F.Cu at (146.8, 156.0)
- added REF**: 1pin, Connect:1pin, F.Cu at (146.8, 124.5)
- added REF**: 1pin, Connect:1pin, F.Cu at (146.8, 92.5)
- C10, C11, C13, C14, C16, C17, C18, C9, R10, R11, R12, R13, R14, R15, R7, R8, R9, U4, U5: moved to F.Cu
- L1: footprint Inductors:self_cms_we-tpc_XL -> v0:CDRH2D14
- R1, R3: moved to B.Cu
- moved L1 61.9 mm to (169.6, 156.2)
- moved U2 58.0 mm to (175.1, 156.9)
- moved C15 57.4 mm to (182.9, 156.5)
- moved C12 52.1 mm to (168.7, 152.1), turned to 180 degrees
- moved P1 44.2 mm to (146.8, 132.0), turned to 270 degrees
- moved U6 39.5 mm to (187.1, 117.1), turned to 0 degrees
- moved C31 33.4 mm to (182.6, 121.0), turned to 90 degrees
- moved C21 30.1 mm to (184.0, 123.6), turned to 180 degrees
- moved C24 21.7 mm to (174.8, 138.0), turned to 270 degrees
- moved IC1 19.0 mm to (147.9, 139.4), turned to 0 degrees
- moved R12 18.0 mm to (166.7, 145.9), turned to 90 degrees
- moved C9 17.5 mm to (166.6, 158.0)
- moved P6 15.1 mm to (189.0, 151.7), turned to 90 degrees
- moved P2 11.8 mm to (200.0, 126.4)
- moved R14 11.3 mm to (174.4, 150.6)
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Connections:
- C31 pad 2: Net-(C31-Pad2) -> GND
- C32 pad 2: Net-(C31-Pad2) -> GND
- U6 pad 1: Net-(C31-Pad2) -> GND
Routing:
- net GND: track 0.00 -> 283.6 mm, vias 0 -> 8
- net +3V3: track 0.00 -> 149.6 mm, vias 0 -> 4
- net /DAT3: track 0.00 -> 55.1 mm, vias 0 -> 3
- net /SD_CLK: track 0.00 -> 53.8 mm, vias 0 -> 3
- net /SD_CONN: track 0.00 -> 53.7 mm, vias 0 -> 3
- net /DAT2: track 0.00 -> 53.5 mm, vias 0 -> 3
- net /SD_CMD: track 0.00 -> 53.3 mm, vias 0 -> 3
- net /xDCS: track 0.00 -> 35.6 mm, vias 0 -> 6
- net /DAT0: track 0.00 -> 30.9 mm, vias 0 -> 3
- net /xRST: track 0.00 -> 30.7 mm, vias 0 -> 2
- net /DAT1: track 0.00 -> 30.2 mm, vias 0 -> 3
- net /DREQ: track 0.00 -> 25.0 mm, vias 0 -> 2
- net Net-(C6-Pad1): track 0.00 -> 24.9 mm, vias 0 -> 2
- net /USB_DM: track 0.00 -> 22.5 mm
- net Net-(R6-Pad1): track 0.00 -> 21.8 mm, vias 0 -> 2
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
Commit message: upd
Parts:
- C26: moved to B.Cu
- R16: footprint Resistors_SMD:R_0603_HandSoldering -> Resistors_SMD:R_1206_HandSoldering
- moved P1 41.6 mm to (162.8, 93.6), turned to 180 degrees
- moved Y3 41.0 mm to (147.0, 131.8), turned to 90 degrees
- moved C19 40.9 mm to (170.7, 92.5)
- moved C3 34.0 mm to (150.9, 134.6)
- moved R7 32.9 mm to (153.1, 149.2), turned to 270 degrees
- moved SW1 32.5 mm to (170.0, 146.9)
- moved L1 32.1 mm to (187.9, 129.8)
- moved C9 30.8 mm to (187.8, 135.7)
- moved C11 27.9 mm to (153.4, 145.1)
- moved R13 26.8 mm to (158.1, 144.5), turned to 0 degrees
- moved U2 26.2 mm to (183.3, 132.1), turned to 90 degrees
- moved R8 25.9 mm to (155.4, 150.9), turned to 270 degrees
- moved U6 25.4 mm to (177.9, 93.5), turned to 90 degrees
- moved C31 24.1 mm to (184.9, 97.0), turned to 270 degrees
- moved C12 23.8 mm to (187.9, 138.0)
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Connections:
- C11 pad 2: Net-(C11-Pad2) -> GND
- C15 pad 2: Net-(C11-Pad2) -> GND
- R11 pad 2: Net-(C11-Pad2) -> GND
- R7 pad 2: Net-(C11-Pad2) -> GND
- R8 pad 2: Net-(C11-Pad2) -> GND
- U4 pad 3: Net-(C11-Pad2) -> GND
Routing:
- net GND: track 283.6 -> 356.3 mm, vias 8 -> 11
- net +3V3: track 149.6 -> 189.4 mm, vias 4 -> 5
- net +BATT: track 0.00 -> 25.5 mm
- net /USB_DM: track 22.5 -> 0.00 mm
- net /USB_DP: track 21.7 -> 0.00 mm
- net /PC4: track 0.00 -> 9.53 mm
- net Net-(P6-Pad1): track 0.00 -> 6.44 mm
- net Net-(L1-Pad1): track 0.00 -> 6.25 mm
- net +5V: track 0.00 -> 5.07 mm
- net Net-(R7-Pad1): track 0.00 -> 4.77 mm
- net /xDCS: track 35.6 -> 30.9 mm, vias 6 -> 4
- net Net-(C14-Pad1): track 0.00 -> 3.83 mm
- net Net-(C14-Pad2): track 0.00 -> 3.65 mm
- net Net-(R8-Pad1): track 0.00 -> 2.75 mm
- net /PC3: track 0.00 -> 1.93 mm
Other:
- net class power added: clearance 0.2, trace_width 0.35, via_dia 0.6, via_drill 0.4

Commit message: pcb of core board v0.01 done!
Parts:
- removed P5: AudioJack, Pin_Headers:Pin_Header_Straight_1x03
- added J1: JACK_TRS_6PINS, v0:ST-033, F.Cu at (153.0, 98.0)
- added SW2: Switch_SPDT_x2, v0:SK22D07-SWITCH, F.Cu at (188.5, 128.8)
- P2: moved to B.Cu
- moved C9 19.4 mm to (188.3, 116.3)
- moved C12 19.4 mm to (188.3, 118.6)
- moved L1 17.9 mm to (188.4, 112.0)
- moved U2 17.9 mm to (183.9, 114.2)
- moved P3 16.7 mm to (159.0, 141.3)
- moved C19 12.0 mm to (182.7, 93.3)
- moved U5 7.58 mm to (174.0, 150.1)
- moved C13 6.61 mm to (178.5, 154.7), turned to 0 degrees
- moved P2 5.97 mm to (185.9, 113.0)
- moved R10 5.88 mm to (168.0, 152.0)
- moved C2 5.46 mm to (150.6, 146.2)
- moved C31 5.00 mm to (180.5, 94.7)
- moved C5 4.43 mm to (170.2, 146.8), turned to 0 degrees
- moved U6 3.43 mm to (174.5, 93.4)
- moved C27 3.31 mm to (172.1, 141.9)
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Connections:
- P2 pad 1: +3V3 -> /I2C2_SDA
- P2 pad 2: GND -> /I2C2_SCL
- P2 pad 3: /PC4 -> /PB2
- P2 pad 4: /PC5 -> /PB1
- P2 pad 5: /PB2 -> /PB0
- P2 pad 6: /PB1 -> /PC5
- P2 pad 7: /PB0 -> /PC4
- P2 pad 8: /I2C2_SCL -> GND
- P2 pad 9: /I2C2_SDA -> +3V3
- P6 pad 2: +BATT -> Net-(P6-Pad2)
Routing:
- net GND: track 356.3 -> 537.5 mm, vias 11 -> 15
- net +3V3: track 189.4 -> 275.4 mm, vias 5 -> 10
- net +5V: track 5.07 -> 86.5 mm, vias 0 -> 2
- net +1V8: track 19.9 -> 83.6 mm, vias 2 -> 6
- net +BATT: track 25.5 -> 85.5 mm, vias 0 -> 3
- net /I2C2_SDA: track 0.00 -> 44.3 mm, vias 0 -> 1
- net /I2C2_SCL: track 0.00 -> 43.6 mm, vias 0 -> 1
- net /PB2: track 0.00 -> 42.5 mm, vias 0 -> 1
- net /USB_DM: track 0.00 -> 41.8 mm, vias 0 -> 2
- net /USB_DP: track 0.00 -> 41.3 mm, vias 0 -> 2
- net /PB1: track 0.00 -> 40.7 mm, vias 0 -> 1
- net /PB0: track 0.00 -> 40.2 mm, vias 0 -> 1
- net /I2C1_SCL: track 12.9 -> 52.0 mm, vias 1 -> 5
- net /I2C1_SDA: track 12.6 -> 48.8 mm, vias 1 -> 5
- net /PC5: track 0.00 -> 35.9 mm, vias 0 -> 1
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- added copper zone on B.Cu, net GND
- added copper zone on F.Cu, net GND
Other:
- net class power removed
- board text added: "SDMPlayer core board v0.01 by Alexander Lutsai 28.04.2016"
- board text added: "https://github.com/SL-RU/sdmplayer"
