File: sch/mplayer/v0.01/sdmplayerv0.01.sch (KiCad schematic (older format))
At the start: 20 parts, among them CON1 SD_Card, IC1 AT24CS64-SSHM, P1 USB_OTG, P2 CONN_01X09, P3 ClockBat, P4 USART1, SW1 SW_PUSH, U1 VS1053, U2 TP4056, U3 STM32F103RCTx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

Commit message: player_scheme_0.01
Parts:
- removed U2: TP4056, SMD_Packages:SO-8_PowerPAK_Vishay_Single, symbol TP4056
- removed X1: 8MHz, symbol CRYSTAL_SMD
- removed X2: 32768Hz, symbol CRYSTAL_SMD
- added C10: 10uF, symbol C
- added C11: 1uF, symbol C
- added C12: 0.47uF, symbol C
- added C13, C14, C18: 0.1uF, symbol C
- added C15: C, symbol C
- added C16, C17: 0.1uF, symbol C_Small
- added C6: 33pF, Capacitors_SMD:C_0805_HandSoldering, symbol C
- added C7: 33pF, Capacitors_SMD:C_0805_HandSoldering, symbol C_Small
- added C8: 1uF, Capacitors_SMD:C_0805_HandSoldering, symbol C
- added C9: 4.7uF, symbol C
- added L1: 2.2uH, symbol L_Small
- added P5: AudioJack, Pin_Headers:Pin_Header_Straight_1x03, symbol CONN_01X03
- added P6: LiPo battery, symbol CONN_01X02
- added R10: 18.2k, symbol R
- added R11: 100k, symbol R
- added R12, R13: 4.7k, symbol R
- added R14, R15: 100, symbol R
- added R16: 0.01, symbol R
- added R4: R, Resistors_SMD:R_0603_HandSoldering, symbol R
- added R5: 1M, Resistors_SMD:R_0603_HandSoldering, symbol R
- added R6: 100k, Resistors_SMD:R_0603_HandSoldering, symbol R
- added R7: 1k, symbol R
- added R8: 2k, symbol R
- added R9: 1.8M, symbol R
- added U2: LM3671MF-3.3, symbol LM3671
- added U4: BQ24090, symbol BQ24090
- added U5: BQ27510, symbol BQ27510
- added Y1: 12.288MHz, Crystals:Crystal_SMD_0603_4Pads, symbol Crystal
- added Y2: 8MHz, Crystals:Crystal_SMD_0603_4Pads, symbol Crystal
- added Y3: 32768Hz, Crystals:Crystal_SMD_0603_4Pads, symbol Crystal
- C1, C2, C3, C4: footprint (none) -> Capacitors_SMD:C_0402
- C5: value C -> 100nF; footprint (none) -> Capacitors_SMD:C_0402
- CON1: footprint Connect:SD_Card_Receptacle -> Housings_SOIC:SOIC-14_3.9x8.7mm_Pitch1.27mm
- IC1: footprint SO8 -> Housings_SOIC:SOIC-8-1EP_3.9x4.9mm_Pitch1.27mm
- P3: footprint (none) -> Pin_Headers:Pin_Header_Straight_1x01
- P4: footprint (none) -> Pin_Headers:Pin_Header_Straight_1x02
- R1, R2, R3: footprint (none) -> Resistors_SMD:R_0603_HandSoldering
- SW1: footprint (none) -> Pin_Headers:Pin_Header_Angled_1x02
Connections:
- net labels added: +1V8, +BATT, DREQ, PA7, PC0, PC1, PC2, PC3, SPI2_MISO, SPI2_MOSI, SPI2_SCK, xCS, xDCS, xRST
- wire segments 82 -> 203
Other:
- note added: "From bat to 3.3V\nBuck converter"
- note added: "Lithium charger\n"
- moved on the sheet: C3, C4, U1

Commit message: fix
Parts:
- added C? (x15): 100nF, symbol C
- added C? (x2): 10uF, symbol CP
- added U?: NCP1117ST18T3G, symbol NCP1117ST18T3G
- C10, C11, C12, C9, L1: footprint (none) -> Capacitors_SMD:C_0805_HandSoldering
- C13, C14, C16, C17, C18: footprint (none) -> Capacitors_SMD:C_1206_HandSoldering
- C15: value C -> 1uF; footprint (none) -> Capacitors_SMD:C_1206_HandSoldering
- P6: footprint (none) -> Socket_Strips:Socket_Strip_Straight_1x02
- R10, R11, R12, R13, R14, R15, R16, R7, R8, R9: footprint (none) -> Resistors_SMD:R_0603_HandSoldering
- U2: footprint (none) -> TO_SOT_Packages_SMD:SOT-23-5
- U4: footprint (none) -> Housings_SSOP:MSOP-10-1EP_3x3mm_Pitch0.5mm
- U5: footprint (none) -> Housings_SSOP:MSOP-12-1EP_3x4mm_Pitch0.65mm
Connections:
- wire segments 203 -> 211
Other:
- note added: "0.01"
- note added: "1.8V converter"
- note added: "MCU board for MDPlayer by Lutsai Alexander"
- note added: "MCU: VS1053\nAUDION CODEC: VS1053"
- note added: "Repository: https://github.com/SL-RU/sdmplayer"

Commit message: fix
Parts:
- gave numbers to parts that had none: 18

Commit message: layout upd
Parts:
- removed C19, C31: 10uF, symbol CP
- removed C33, C34, C35: 100nF, symbol C
- removed R4: R, Resistors_SMD:R_0603_HandSoldering, symbol R
- added C19: 10uF, Capacitors_SMD:C_0805_HandSoldering, symbol C
- added C31: 100nF, Capacitors_SMD:C_0402, symbol C
- C11, C8: footprint Capacitors_SMD:C_0805_HandSoldering -> Capacitors_SMD:C_0603_HandSoldering
- C13, C14, C16, C17, C18: footprint Capacitors_SMD:C_1206_HandSoldering -> Capacitors_SMD:C_0402
- C15: footprint Capacitors_SMD:C_1206_HandSoldering -> Capacitors_SMD:C_0603_HandSoldering
- C20, C21, C22, C23, C24, C25, C26, C27, C28, C29, C30, C32: footprint (none) -> Capacitors_SMD:C_0402
- CON1: footprint Housings_SOIC:SOIC-14_3.9x8.7mm_Pitch1.27mm -> v0:Micro_SD_card_slot
- L1: footprint Capacitors_SMD:C_0805_HandSoldering -> Inductors:self_cms_we-tpc_XL
- SW1: footprint Pin_Headers:Pin_Header_Angled_1x02 -> Pin_Headers:Pin_Header_Straight_1x02
- U5: footprint Housings_SSOP:MSOP-12-1EP_3x4mm_Pitch0.65mm -> v0:SON-12
- U6: footprint (none) -> TO_SOT_Packages_SMD:SOT-223
- Y1, Y2: footprint Crystals:Crystal_SMD_0603_4Pads -> Crystals:Crystal_HC49-SD_SMD
- Y3: footprint Crystals:Crystal_SMD_0603_4Pads -> v0:KX-327S
Connections:
- wire segments 211 -> 210

Commit message: upd
Parts:
- L1: footprint Inductors:self_cms_we-tpc_XL -> v0:CDRH2D14
Connections:
- wire segments 210 -> 211
Changed lines of the file:
@@
 F 0 "L1" H 1830 5840 50  0000 L CNN
 F 1 "2.2uH" H 1830 5760 50  0000 L CNN
-F 2 "Inductors:self_cms_we-tpc_XL" H 1800 5800 50  0001 C CNN
+F 2 "v0:CDRH2D14" H 1800 5800 50  0001 C CNN
 F 3 "" H 1800 5800 50  0000 C CNN
 	1    1800 5800
@@
 Wire Wire Line
 	6850 5400 6150 5400
+$Comp
+L GND #PWR038
+U 1 1 571BF1BE
+P 6500 5500
+F 0 "#PWR038" H 6500 5250 50  0001 C CNN
+F 1 "GND" H 6500 5350 50  0000 C CNN
+F 2 "" H 6500 5500 50  0000 C CNN
+F 3 "" H 6500 5500 50  0000 C CNN
+	1    6500 5500
+	1    0    0    -1
+$EndComp
+Wire Wire Line
+	6500 5400 6500 5500
+Connection ~ 6500 5400
 $EndSCHEMATC

Commit message: upd
Parts:
- R16: footprint Resistors_SMD:R_0603_HandSoldering -> Resistors_SMD:R_1206_HandSoldering
Changed lines of the file:
@@
 F 0 "R16" V 5380 6350 50  0000 C CNN
 F 1 "0.01" V 5300 6350 50  0000 C CNN
-F 2 "Resistors_SMD:R_0603_HandSoldering" V 5230 6350 50  0001 C CNN
+F 2 "Resistors_SMD:R_1206_HandSoldering" V 5230 6350 50  0001 C CNN
 F 3 "" H 5300 6350 50  0000 C CNN
 	1    5300 6350
@@
 $EndComp
 Wire Wire Line
-	4850 7600 4850 7600
+	4600 7600 4850 7600
 Connection ~ 4850 7000
 Connection ~ 4850 7600
@@
 	6500 5400 6500 5500
 Connection ~ 6500 5400
+Connection ~ 4600 7600
 $EndSCHEMATC

Commit message: pcb of core board v0.01 done!
Parts:
- removed P5: AudioJack, Pin_Headers:Pin_Header_Straight_1x03, symbol CONN_01X03
- added J1: JACK_TRS_6PINS, v0:ST-033, symbol JACK_TRS_6PINS
- added SW2: Switch_SPDT_x2, v0:SK22D07-SWITCH, symbol Switch_SPDT_x2
Connections:
- wire segments 211 -> 220

Commit message: fix
Parts:
- added C33: 100pF, Capacitors_SMD:C_0805_HandSoldering, symbol C_Small
- added P5: CONN_01X03, Socket_Strips:Socket_Strip_Straight_1x03, symbol CONN_01X03
- added P7, P8: gnd, Socket_Strips:Socket_Strip_Straight_1x01, symbol CONN_01X01
- added P9: 3.3v, Socket_Strips:Socket_Strip_Straight_1x01, symbol CONN_01X01
Connections:
- net labels added: SWCLK, SWDIO
- wire segments 220 -> 229
Changed lines of the file:
@@
 L GND #PWR014
 U 1 1 5715EB9A
-P 7500 6050
-F 0 "#PWR014" H 7500 5800 50  0001 C CNN
-F 1 "GND" H 7500 5900 50  0000 C CNN
-F 2 "" H 7500 6050 50  0000 C CNN
-F 3 "" H 7500 6050 50  0000 C CNN
-	1    7500 6050
+P 7500 6100
+F 0 "#PWR014" H 7500 5850 50  0001 C CNN
+F 1 "GND" H 7500 5950 50  0000 C CNN
+F 2 "" H 7500 6100 50  0000 C CNN
+F 3 "" H 7500 6100 50  0000 C CNN
+	1    7500 6100
 	1    0    0    -1
 $EndComp
@@
 	8700 5600 8600 5600
 Connection ~ 8600 5700
-Wire Bus Line
-	3850 700  3850 4950
 Wire Wire Line
 	3950 4200 4900 4200
@@
 	2350 7050 2900 7050
 Wire Wire Line
-	2350 7700 4600 7700
+	4600 7700 2350 7700
 Wire Wire Line
 	2350 7000 2350 7200
 Connection ~ 2350 7050
 Wire Wire Line
-	2350 7500 2350 7700
+	2350 7700 2350 7500
 Wire Wire Line
 	2900 7150 2600 7150
@@
 Connection ~ 4600 7050
 Wire Wire Line
-	4600 7700 4600 7500
+	4600 7500 4600 7700
 Connection ~ 4400 7700
 Wire Notes Line
@@
 Connection ~ 2250 4950
 Wire Wire Line
-	2050 5300 2050 5250
+	2050 5250 2050 5300
 Connection ~ 2050 5250
 Wire Wire Line
@@
 Connection ~ 1400 5250
 Wire Wire Line
-	3650 4950 1400 4950
-Wire Wire Line
-	1400 5250 3650 5250
+	1400 4950 3950 4950
+Wire Wire Line
+	950  5250 3650 5250
 Connection ~ 800  2800
 Wire Wire Line
-	6850 5050 6850 5100
-Wire Wire Line
-	6850 5100 6550 5100
-Wire Wire Line
-	6850 5400 6150 5400
+	6850 5100 6850 5050
+Wire Wire Line
+	6550 5100 6850 5100
+Wire Wire Line
+	6150 5400 6850 5400
 Wire Wire Line
 	6500 5400 6500 5500
@@
 Connection ~ 4600 7600
 Wire Wire Line
-	7500 6050 7500 6000
+	7500 6000 7500 6100
 Wire Wire Line
 	2600 6000 2700 6000
@@
 Wire Wire Line
 	2850 5550 2850 6000
+$Comp
+L CONN_01X03 P5
+U 1 1 572F829A
+P 7900 5750
+F 0 "P5" H 7900 5950 50  0000 C CNN
+F 1 "CONN_01X03" V 8000 5750 50  0000 C CNN
+F 2 "Socket_Strips:Socket_Strip_Straight_1x03" H 7900 5750 50  0001 C CNN
+F 3 "" H 7900 5750 50  0000 C CNN
+	1    7900 5750
+	0    -1   -1   0
+$EndComp
+Entry Wire Line
+	7900 6400 8000 6500
+Entry Wire Line
+	8000 6400 8100 6500
+Wire Wire Line
+	8000 6400 8000 5950
+Wire Wire Line
+	7900 5950 7900 6400
+Wire Wire Line
+	7800 5950 7800 6250
+Wire Wire Line
+	7800 6250 7650 6250
+Wire Wire Line
+	7650 6050 7650 6350
+Wire Wire Line
+	7650 6050 7500 6050
+Connection ~ 7500 6050
+Text Label 7900 6250 1    60   ~ 0
+SWCLK
+Text Label 8000 6250 1    60   ~ 0
+SWDIO
+Text Label 10850 2700 2    60   ~ 0
+SWCLK
+Wire Wire Line
+	10500 2700 11050 2700
+Wire Wire Line
+	10500 2600 11050 2600
+Text Label 10550 2600 0    60   ~ 0
+SWDIO
+Entry Wire Line
+	11050 2600 11150 2700
+Entry Wire Line
+	11050 2700 11150 2800
+$Comp
+L C_Small C33
+U 1 1 572FDE6D
+P 7750 6350
+F 0 "C33" H 7760 6420 50  0000 L CNN
+F 1 "100pF" H 7760 6270 50  0000 L CNN
+F 2 "Capacitors_SMD:C_0805_HandSoldering" H 7750 6350 50  0001 C CNN
+F 3 "" H 7750 6350 50  0000 C CNN
+	1    7750 6350
+	0    1    1    0
+$EndComp
+Wire Wire Line
+	7850 6350 7900 6350
+Connection ~ 7900 6350
+Connection ~ 7650 6250
+$Comp
+L CONN_01X01 P8
+U 1 1 57310A61
+P 1200 5050
+F 0 "P8" H 1200 5150 50  0000 C CNN
+F 1 "gnd" V 1300 5050 50  0000 C CNN
+F 2 "Socket_Strips:Socket_Strip_Straight_1x01" H 1200 5050 50  0001 C CNN
+F 3 "" H 1200 5050 50  0000 C CNN
+	1    1200 5050
+	0    -1   -1   0
+$EndComp
+$Comp
+L CONN_01X01 P7
+U 1 1 57310B20
+P 950 5050
+F 0 "P7" H 950 5150 50  0000 C CNN
+F 1 "gnd" V 1050 5050 50  0000 C CNN
+F 2 "Socket_Strips:Socket_Strip_Straight_1x01" H 950 5050 50  0001 C CNN
+F 3 "" H 950 5050 50  0000 C CNN
+	1    950  5050
+	0    -1   -1   0
+$EndComp
+Connection ~ 1200 5250
+$Comp
+L CONN_01X01 P9
+U 1 1 57312373
+P 3950 5150
+F 0 "P9" H 3950 5250 50  0000 C CNN
+F 1 "3.3v" V 4050 5150 50  0000 C CNN
+F 2 "Socket_Strips:Socket_Strip_Straight_1x01" H 3950 5150 50  0001 C CNN
+F 3 "" H 3950 5150 50  0000 C CNN
+	1    3950 5150
+	0    1    1    0
+$EndComp
+Wire Bus Line
+	3850 4350 3850 700
+Connection ~ 3650 4950
 $EndSCHEMATC
